File: board/Bar.kicad_pcb (KiCad board)
At the start: 2 copper layers, 55 x 80 mm, 28 parts, among them J1 SUPPLY, J2 SUPPLY, J3 USB_A, J4 Screw_Terminal_01x02, J5 SUPPLY, J6 SUPPLY, U1 74HC595, U2 74HC595, U3 ATtiny85-20PU

Commit message: added leds for representing the mode added first version of the software
Parts:
- added D1: LED, LED_SMD:LED_1206_3216Metric_Pad1.42x1.75mm_HandSolder, F.Cu at (63.5, 81.3)
- added D2: LED, LED_SMD:LED_1206_3216Metric_Pad1.42x1.75mm_HandSolder, F.Cu at (63.7, 70.6)
- added D3: LED, LED_SMD:LED_1206_3216Metric_Pad1.42x1.75mm_HandSolder, F.Cu at (63.7, 74.2)
- added D4: LED, LED_SMD:LED_1206_3216Metric_Pad1.42x1.75mm_HandSolder, F.Cu at (63.5, 77.7)
- added D5: LED, LED_SMD:LED_1206_3216Metric_Pad1.42x1.75mm_HandSolder, F.Cu at (63.5, 67.1)
- added D6: LED, LED_SMD:LED_1206_3216Metric_Pad1.42x1.75mm_HandSolder, F.Cu at (63.7, 63.5)
- added R11: 100, Resistor_SMD:R_0805_2012Metric_Pad1.15x1.40mm_HandSolder, F.Cu at (64.4, 60.3)
- added R12: 100, Resistor_SMD:R_0805_2012Metric_Pad1.15x1.40mm_HandSolder, F.Cu at (58.9, 82.9)
- added R13: 100, Resistor_SMD:R_0805_2012Metric_Pad1.15x1.40mm_HandSolder, F.Cu at (56.3, 89.7)
- added R14: 100, Resistor_SMD:R_0805_2012Metric_Pad1.15x1.40mm_HandSolder, F.Cu at (62.9, 36.1)
- added R15: 100, Resistor_SMD:R_0805_2012Metric_Pad1.15x1.40mm_HandSolder, F.Cu at (62.2, 29.1)
- added R16: 100, Resistor_SMD:R_0805_2012Metric_Pad1.15x1.40mm_HandSolder, F.Cu at (64.8, 44.6)
- added RV2: R_POT, Potentiometer_THT:Potentiometer_ACP_CA6-H2,5_Horizontal, F.Cu at (47.8, 16.3)
- C1, C2, C3: value 100µ -> 100nF
Connections:
- U1 pad 2: Net-(U1-Pad2) -> /OUT_1
- U1 pad 3: Net-(U1-Pad3) -> /OUT_2
- U1 pad 4: Net-(U1-Pad4) -> /OUT_3
- U1 pad 5: Net-(U1-Pad5) -> /OUT_4
- U1 pad 6: Net-(U1-Pad6) -> /OUT_5
- U1 pad 7: Net-(U1-Pad7) -> /OUT_6
- U3 pad 3: Net-(U3-Pad3) -> /MODE

Commit message: final board
Parts:
- removed the J3 at (8.26, 29.2)
- added J3 (x3): USB_A, myfootprint:LUM_2410_06_USB_A_SMD, F.Cu at (15.5, 36.6)
- RV2: footprint Potentiometer_THT:Potentiometer_ACP_CA6-H2,5_Horizontal -> Potentiometer_THT:Potentiometer_Piher_PT-10-V10_Vertical
- moved RV2 72.8 mm to (50.8, 89.0), turned to 270 degrees
- moved R15 51.6 mm to (64.5, 80.6)
- moved J4 49.6 mm to (63.9, 89.2), turned to 270 degrees
- moved R16 40.4 mm to (64.5, 85.0)
- moved R14 40.3 mm to (64.5, 76.3)
- moved D6 21.8 mm to (59.7, 85.0), turned to 180 degrees
- moved R13 19.8 mm to (64.5, 71.6)
- moved D1 19.5 mm to (59.7, 62.2), turned to 180 degrees
- moved R12 16.9 mm to (64.5, 66.9)
- moved D5 14.1 mm to (59.7, 80.6), turned to 180 degrees
- moved REF** 11.2 mm to (22.0, 97.1)
- moved C3 10.5 mm to (41.8, 79.4), turned to 270 degrees
- moved REF** 10.0 mm to (61.9, 97.5)
- moved J6 9.43 mm to (44.1, 95.1)
- moved RV1 8.04 mm to (31.4, 73.5)
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Connections:
- J4 pad 2: GND -> /MODE
- U3 pad 6: /CLOCK -> /DATA
- U3 pad 7: /DATA -> /CLOCK
Routing:
- net /OUT_6: track 0.00 -> 27.7 mm, vias 0 -> 2
- net /MODE: track 0.00 -> 25.1 mm
- net /OUT_5: track 0.00 -> 22.6 mm, vias 0 -> 2
- net /OUT_4: track 0.00 -> 16.7 mm
- net /OUT_1: track 0.00 -> 13.3 mm, vias 0 -> 2
- net /OUT_3: track 0.00 -> 12.0 mm
- net /OUT_2: track 0.00 -> 8.79 mm
- net /SHIFT_OUT: track 17.1 -> 23.9 mm
- net +5V: track 205.4 -> 203.0 mm
- net Net-(D5-Pad1): track 0.00 -> 2.31 mm
- net Net-(D6-Pad1): track 0.00 -> 2.31 mm
- net Net-(D4-Pad1): track 0.00 -> 2.31 mm
- net Net-(D3-Pad1): track 0.00 -> 2.31 mm
- net Net-(D2-Pad1): track 0.00 -> 2.31 mm
- net Net-(D1-Pad1): track 0.00 -> 2.31 mm
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Other:
- board size 55 x 80 mm -> 50 x 90 mm
- board text added: "01/2019"
- board text added: "1"
- board text added: "10"
- board text added: "2"
- board text added: "3"
- board text added: "4"
- board text added: "5"
- board text added: "5V"
- board text added: "6"
- board text added: "7"
- board text added: "8"
- board text added: "9"
- board text added: "MODE"
- board text added: "MODE-1"
- board text added: "MODE-2"
- board text added: "MODE-3"
- board text added: "MODE-4"
- board text added: "MODE-5"
- board text added: "MODE-6"
- board text added: "Select mode"
- board text added: "Select value"
- board text added: "Slide-O-Bar V1.0"
- board text added: "VALUE"
- board text removed: "+"
